Commit message: fixing starting pos

File: src/my_arm_description/urdf/my_arm.urdf.xacro (robot description, xacro)
@@ -111,28 +111,3 @@
     <limit lower="-3.14" upper="3.14" effort="50" velocity="2.0"/>
   </joint>
-  <ros2_control name="MyRobotSystem" type="system">
-    <hardware>
-        <plugin>mock_components/GenericSystem</plugin>
-    </hardware>
-    <joint name="joint_1">
-      <command_interface name="position"/>
-      <state_interface name="position"/>
-      <state_interface name="velocity"/>
-    </joint>
-    <joint name="joint_2">
-      <command_interface name="position"/>
-      <state_interface name="position"/>
-      <state_interface name="velocity"/>
-    </joint>
-    <joint name="joint_3">
-      <command_interface name="position"/>
-      <state_interface name="position"/>
-      <state_interface name="velocity"/>
-    </joint>
-    <joint name="joint_4">
-      <command_interface name="position"/>
-      <state_interface name="position"/>
-      <state_interface name="velocity"/>
-    </joint>
-  </ros2_control>
 </robot>

File: src/my_arm_moveit_config/config/my_arm.ros2_control.xacro (robot description, xacro)
@@ -2,5 +2,5 @@
 <robot xmlns:xacro="http://www.ros.org/wiki/xacro">
     <xacro:macro name="my_arm_ros2_control" params="name initial_positions_file">
-        <xacro:property name="initial_positions" value="${load_yaml(initial_positions_file)['initial_positions']}"/>
+        <xacro:property name="initial_positions" value="${xacro.load_yaml(initial_positions_file)['initial_positions']}"/>
         <ros2_control name="${name}" type="system">
             <hardware>
@@ -13,4 +13,5 @@
                   <param name="initial_value">${initial_positions['joint_1']}</param>
                 </state_interface>
+                <state_interface name="velocity"/>
             </joint>
             <joint name="joint_2">
@@ -19,4 +20,5 @@
                   <param name="initial_value">${initial_positions['joint_2']}</param>
                 </state_interface>
+                <state_interface name="velocity"/>
             </joint>
             <joint name="joint_3">
@@ -25,4 +27,5 @@
                   <param name="initial_value">${initial_positions['joint_3']}</param>
                 </state_interface>
+                <state_interface name="velocity"/>
             </joint>
             <joint name="joint_4">
@@ -31,4 +34,5 @@
                   <param name="initial_value">${initial_positions['joint_4']}</param>
                 </state_interface>
+                <state_interface name="velocity"/>
             </joint>
         </ros2_control>

File: src/my_arm_moveit_config/config/my_arm.urdf.xacro (robot description, xacro)
@@ -1,5 +1,5 @@
 <?xml version="1.0"?>
 <robot xmlns:xacro="http://www.ros.org/wiki/xacro" name="my_arm">
-    <xacro:arg name="initial_positions_file" default="initial_positions.yaml" />
+    <xacro:arg name="initial_positions_file" default="$(find my_arm_moveit_config)/config/initial_positions.yaml" />
     <!-- Import my_arm urdf file -->
     <xacro:include filename="$(find my_arm_description)/urdf/my_arm.urdf.xacro" />

Commit message: Full simulation working except gripper open and close

File: src/my_arm_description/urdf/my_arm.urdf.xacro (robot description, xacro)
@@ -83,4 +83,49 @@
     </collision>
   </link>
+  <link name="link_5">
+    <visual>
+      <geometry>
+        <cylinder length="0.02" radius="0.03"/>
+      </geometry>
+      <origin xyz="0 0 0.01" rpy="0 0 0"/>
+      <material name="blue"/>
+    </visual>
+    <collision>
+      <geometry>
+        <cylinder length="0.02" radius="0.03"/>
+      </geometry>
+      <origin xyz="0 0 0.01" rpy="0 0 0"/>
+    </collision>
+  </link>
+  <link name="left_finger">
+    <visual>
+      <geometry>
+        <box size="0.01 0.01 0.06"/>
+      </geometry>
+      <origin xyz="0 0 0.03" rpy="0 0 0"/>
+      <material name="orange"/>
+    </visual>
+    <collision>
+      <geometry>
+        <box size="0.01 0.01 0.06"/>
+      </geometry>
+      <origin xyz="0 0 0.03" rpy="0 0 0"/>
+    </collision>
+  </link>
+  <link name="right_finger">
+    <visual>
+      <geometry>
+        <box size="0.01 0.01 0.06"/>
+      </geometry>
+      <origin xyz="0 0 0.03" rpy="0 0 0"/>
+      <material name="orange"/>
+    </visual>
+    <collision>
+      <geometry>
+        <box size="0.01 0.01 0.06"/>
+      </geometry>
+      <origin xyz="0 0 0.03" rpy="0 0 0"/>
+    </collision>
+  </link>
   <joint name="joint_1" type="revolute">
     <parent link="base_link"/>
@@ -97,5 +142,5 @@
     <limit lower="-1.57" upper="1.57" effort="200" velocity="0.6"/>
   </joint>
-<joint name="joint_3" type="revolute">
+  <joint name="joint_3" type="revolute">
     <parent link="link_2"/>
     <child link="link_3"/>
@@ -111,3 +156,25 @@
     <limit lower="-3.14" upper="3.14" effort="50" velocity="2.0"/>
   </joint>
+  <joint name="joint_5" type="revolute">
+    <parent link="link_4"/>
+    <child link="link_5"/>
+    <origin xyz="0 0 0.05" rpy="0 0 0"/>
+    <axis xyz="0 0 1"/>
+    <limit lower="-3.14" upper="3.14" effort="50" velocity="2.0"/>
+  </joint>
+  <joint name="gripper_joint" type="prismatic">
+    <parent link="link_5"/>
+    <child link="left_finger"/>
+    <origin xyz="0 0.015 0.02" rpy="0 0 0"/>
+    <axis xyz="0 1 0"/>
+    <limit lower="0.0" upper="0.03" effort="20" velocity="0.5"/>
+  </joint>
+  <joint name="right_finger_joint" type="prismatic">
+    <parent link="link_5"/>
+    <child link="right_finger"/>
+    <origin xyz="0 -0.015 0.02" rpy="0 0 0"/>
+    <axis xyz="0 -1 0"/>
+    <limit lower="0.0" upper="0.03" effort="20" velocity="0.5"/>
+    <mimic joint="gripper_joint" multiplier="1.0"/>
+  </joint>
 </robot>

File: src/my_arm_moveit_config/config/my_arm.ros2_control.xacro (robot description, xacro)
@@ -36,4 +36,18 @@
                 <state_interface name="velocity"/>
             </joint>
+            <joint name="joint_5">
+                <command_interface name="position"/>
+                <state_interface name="position">
+                  <param name="initial_value">${initial_positions['joint_5']}</param>
+                </state_interface>
+                <state_interface name="velocity"/>
+            </joint>
+            <joint name="gripper_joint">
+                <command_interface name="position"/>
+                <state_interface name="position">
+                  <param name="initial_value">${initial_positions['gripper_joint']}</param>
+                </state_interface>
+                <state_interface name="velocity"/>
+            </joint>
         </ros2_control>
     </xacro:macro>

Commit message: Moveit arm works

File: src/my_arm_description/urdf/my_arm.urdf.xacro (robot description, xacro)
@@ -1,4 +1,7 @@
 <?xml version="1.0"?>
 <robot xmlns:xacro="http://www.ros.org/wiki/xacro" name="my_arm">
+  <xacro:arg name="use_mock_hardware" default="false" />
+  <xacro:arg name="include_ros2_control" default="false" />
+  <xacro:property name="use_mock" value="$(arg use_mock_hardware)"/>
   <material name="blue">
     <color rgba="0 0 0.8 1"/>
@@ -41,14 +44,14 @@
     <visual>
       <geometry>
-        <cylinder length="0.4" radius="0.025"/>
+        <cylinder length="0.405" radius="0.025"/>
       </geometry>
-      <origin xyz="0 0 0.2" rpy="0 0 0"/>
+      <origin xyz="0 0 0.2025" rpy="0 0 0"/>
       <material name="orange"/>
     </visual>
     <collision>
       <geometry>
-        <cylinder length="0.4" radius="0.025"/>
+        <cylinder length="0.405" radius="0.025"/>
       </geometry>
-      <origin xyz="0 0 0.2" rpy="0 0 0"/>
+      <origin xyz="0 0 0.2025" rpy="0 0 0"/>
     </collision>
   </link>
@@ -56,14 +59,14 @@
     <visual>
       <geometry>
-        <cylinder length="0.4" radius="0.015"/>
+        <cylinder length="0.345" radius="0.015"/>
       </geometry>
-      <origin xyz="0 0 0.2" rpy="0 0 0"/>
+      <origin xyz="0 0 0.1725" rpy="0 0 0"/>
       <material name="blue"/>
     </visual>
     <collision>
       <geometry>
-        <cylinder length="0.4" radius="0.015"/>
+        <cylinder length="0.345" radius="0.015"/>
       </geometry>
-      <origin xyz="0 0 0.2" rpy="0 0 0"/>
+      <origin xyz="0 0 0.1725" rpy="0 0 0"/>
     </collision>
   </link>
@@ -88,5 +91,5 @@
     <origin xyz="0 0 0.025" rpy="0 0 0"/>
     <axis xyz="0 0 1"/>
-    <limit lower="-3.14" upper="3.14" effort="100" velocity="1.0"/>
+    <limit lower="0.0" upper="6.283185" effort="100" velocity="1.0"/>
   </joint>
   <joint name="joint_2" type="revolute">
@@ -95,44 +98,72 @@
     <origin xyz="0 0 0.1" rpy="0 0 0"/>
     <axis xyz="0 1 0"/>
-    <limit lower="-1.57" upper="1.57" effort="200" velocity="0.6"/>
+    <limit lower="-1.570796" upper="1.221730" effort="200" velocity="0.6"/>
   </joint>
-<joint name="joint_3" type="revolute">
+  <joint name="joint_3" type="revolute">
     <parent link="link_2"/>
     <child link="link_3"/>
-    <origin xyz="0 0 0.4" rpy="0 0 0"/>
+    <origin xyz="0 0 0.405" rpy="0 0 0"/>
     <axis xyz="0 1 0"/>
-    <limit lower="-2.5" upper="2.5" effort="100" velocity="0.26"/>
+    <limit lower="-3.141593" upper="0.0" effort="100" velocity="0.26"/>
   </joint>
   <joint name="joint_4" type="revolute">
     <parent link="link_3"/>
     <child link="link_4"/>
-    <origin xyz="0 0 0.4" rpy="0 0 0"/>
+    <origin xyz="0 0 0.345" rpy="0 0 0"/>
     <axis xyz="0 1 0"/>
     <limit lower="-3.14" upper="3.14" effort="50" velocity="2.0"/>
   </joint>
-  <ros2_control name="MyRobotSystem" type="system">
-    <hardware>
-        <plugin>mock_components/GenericSystem</plugin>
-    </hardware>
-    <joint name="joint_1">
-      <command_interface name="position"/>
-      <state_interface name="position"/>
-      <state_interface name="velocity"/>
-    </joint>
-    <joint name="joint_2">
-      <command_interface name="position"/>
-      <state_interface name="position"/>
-      <state_interface name="velocity"/>
-    </joint>
-    <joint name="joint_3">
-      <command_interface name="position"/>
-      <state_interface name="position"/>
-      <state_interface name="velocity"/>
-    </joint>
-    <joint name="joint_4">
-      <command_interface name="position"/>
-      <state_interface name="position"/>
-      <state_interface name="velocity"/>
-    </joint>
-  </ros2_control>
+  <xacro:if value="$(arg include_ros2_control)">
+    <ros2_control name="MyRobotSystem" type="system">
+      <hardware>
+          <xacro:if value="${use_mock}">
+            <plugin>mock_components/GenericSystem</plugin>
+          </xacro:if>
+          <xacro:unless value="${use_mock}">
+            <plugin>my_arm_hardware/Esp32SerialHardware</plugin>
+            <param name="port">/dev/ttyUSB0</param>
+            <param name="baud_rate">115200</param>
+            <param name="real_joints">3</param>
+            <param name="id_offset">0</param>
+            <param name="query_period_ms">50</param>
+            <param name="poll_cur_ang">false</param>
+            <param name="stream_list_mode">true</param>
+            <param name="stream_without_id">false</param>
+            <param name="wait_for_first_state">true</param>
+            <param name="state_timeout_ms">1000</param>
+            <param name="ping_on_activate">true</param>
+            <param name="ping_id">50</param>
+            <param name="ping_timeout_ms">300</param>
+            <param name="joint_1_min_deg">0</param>
+            <param name="joint_1_max_deg">360</param>
+            <param name="joint_2_min_deg">0</param>
+            <param name="joint_2_max_deg">160</param>
+            <param name="joint_1_offset_deg">0</param>
+            <param name="joint_2_offset_deg">-90</param>
+            <param name="joint_3_offset_deg">-90</param>
+            <param name="joint_4_offset_deg">0</param>
+          </xacro:unless>
+      </hardware>
+      <joint name="joint_1">
+        <command_interface name="position"/>
+        <state_interface name="position"/>
+        <state_interface name="velocity"/>
+      </joint>
+      <joint name="joint_2">
+        <command_interface name="position"/>
+        <state_interface name="position"/>
+        <state_interface name="velocity"/>
+      </joint>
+      <joint name="joint_3">
+        <command_interface name="position"/>
+        <state_interface name="position"/>
+        <state_interface name="velocity"/>
+      </joint>
+      <joint name="joint_4">
+        <command_interface name="position"/>
+        <state_interface name="position"/>
+        <state_interface name="velocity"/>
+      </joint>
+    </ros2_control>
+  </xacro:if>
 </robot>

File: src/my_arm_moveit_config/config/my_arm.ros2_control.xacro (robot description, xacro)
@@ -1,10 +1,36 @@
 <?xml version="1.0"?>
 <robot xmlns:xacro="http://www.ros.org/wiki/xacro">
-    <xacro:macro name="my_arm_ros2_control" params="name initial_positions_file">
+    <xacro:macro name="my_arm_ros2_control" params="name initial_positions_file use_mock_hardware">
         <xacro:property name="initial_positions" value="${load_yaml(initial_positions_file)['initial_positions']}"/>
+      <xacro:property name="use_mock" value="${use_mock_hardware}"/>
         <ros2_control name="${name}" type="system">
             <hardware>
-                <!-- By default, set up controllers for simulation. This won't work on real hardware -->
-                <plugin>mock_components/GenericSystem</plugin>
+          <xacro:if value="${use_mock}">
+            <plugin>mock_components/GenericSystem</plugin>
+          </xacro:if>
+          <xacro:unless value="${use_mock}">
+            <plugin>my_arm_hardware/Esp32SerialHardware</plugin>
+            <param name="port">/dev/ttyUSB0</param>
+            <param name="baud_rate">115200</param>
+                    <param name="real_joints">3</param>
+                    <param name="id_offset">0</param>
+            <param name="query_period_ms">50</param>
+                    <param name="poll_cur_ang">false</param>
+                    <param name="stream_list_mode">true</param>
+                    <param name="stream_without_id">false</param>
+                    <param name="wait_for_first_state">true</param>
+                    <param name="state_timeout_ms">1000</param>
+            <param name="ping_on_activate">true</param>
+                    <param name="ping_id">50</param>
+            <param name="ping_timeout_ms">300</param>
+            <param name="joint_1_min_deg">0</param>
+            <param name="joint_1_max_deg">360</param>
+            <param name="joint_2_min_deg">0</param>
+            <param name="joint_2_max_deg">160</param>
+            <param name="joint_1_offset_deg">0</param>
+            <param name="joint_2_offset_deg">-90</param>
+            <param name="joint_3_offset_deg">-90</param>
+            <param name="joint_4_offset_deg">0</param>
+          </xacro:unless>
             </hardware>
             <joint name="joint_1">
@@ -13,4 +39,5 @@
                   <param name="initial_value">${initial_positions['joint_1']}</param>
                 </state_interface>
+                <state_interface name="velocity"/>
             </joint>
             <joint name="joint_2">
@@ -19,4 +46,5 @@
                   <param name="initial_value">${initial_positions['joint_2']}</param>
                 </state_interface>
+                <state_interface name="velocity"/>
             </joint>
             <joint name="joint_3">
@@ -25,4 +53,5 @@
                   <param name="initial_value">${initial_positions['joint_3']}</param>
                 </state_interface>
+                <state_interface name="velocity"/>
             </joint>
             <joint name="joint_4">
@@ -31,4 +60,5 @@
                   <param name="initial_value">${initial_positions['joint_4']}</param>
                 </state_interface>
+                <state_interface name="velocity"/>
             </joint>
         </ros2_control>

File: src/my_arm_moveit_config/config/my_arm.urdf.xacro (robot description, xacro)
@@ -2,8 +2,12 @@
 <robot xmlns:xacro="http://www.ros.org/wiki/xacro" name="my_arm">
     <xacro:arg name="initial_positions_file" default="initial_positions.yaml" />
+    <xacro:arg name="use_mock_hardware" default="false" />
     <!-- Import my_arm urdf file -->
     <xacro:include filename="$(find my_arm_description)/urdf/my_arm.urdf.xacro" />
     <!-- Import control_xacro -->
     <xacro:include filename="my_arm.ros2_control.xacro" />
-    <xacro:my_arm_ros2_control name="FakeSystem" initial_positions_file="$(arg initial_positions_file)"/>
+    <xacro:my_arm_ros2_control
+        name="FakeSystem"
+        initial_positions_file="$(arg initial_positions_file)"
+        use_mock_hardware="$(arg use_mock_hardware)"/>
 </robot>

Commit message: broken

File: src/my_arm_description/urdf/my_arm.urdf.xacro (robot description, xacro)
@@ -3,4 +3,6 @@
   <xacro:arg name="use_mock_hardware" default="false" />
   <xacro:arg name="include_ros2_control" default="false" />
+  <xacro:arg name="initial_positions_file" default="$(find-pkg-share my_arm_moveit_config)/config/initial_positions.yaml" />
+  <xacro:property name="initial_positions_file" value="$(arg initial_positions_file)"/>
   <xacro:property name="use_mock" value="$(arg use_mock_hardware)"/>
   <material name="blue">
@@ -86,10 +88,10 @@
     </collision>
   </link>
-  <joint name="joint_1" type="revolute">
+  <joint name="joint_1" type="continuous">
     <parent link="base_link"/>
     <child link="link_1"/>
     <origin xyz="0 0 0.025" rpy="0 0 0"/>
     <axis xyz="0 0 1"/>
-    <limit lower="0.0" upper="6.283185" effort="100" velocity="1.0"/>
+    <limit effort="100" velocity="1.0"/>
   </joint>
   <joint name="joint_2" type="revolute">
@@ -98,5 +100,5 @@
     <origin xyz="0 0 0.1" rpy="0 0 0"/>
     <axis xyz="0 1 0"/>
-    <limit lower="-1.570796" upper="1.221730" effort="200" velocity="0.6"/>
+    <limit lower="-1.570796" upper="1.221730" effort="200" velocity="0.45"/>
   </joint>
   <joint name="joint_3" type="revolute">
@@ -105,5 +107,5 @@
     <origin xyz="0 0 0.405" rpy="0 0 0"/>
     <axis xyz="0 1 0"/>
-    <limit lower="-3.141593" upper="0.0" effort="100" velocity="0.26"/>
+    <limit lower="-3.141593" upper="0.0" effort="100" velocity="1.35"/>
   </joint>
   <joint name="joint_4" type="revolute">
@@ -115,4 +117,7 @@
   </joint>
   <xacro:if value="$(arg include_ros2_control)">
+    <xacro:if value="${use_mock}">
+      <xacro:property name="initial_positions" value="${xacro.load_yaml(initial_positions_file)['initial_positions']}"/>
+    </xacro:if>
     <ros2_control name="MyRobotSystem" type="system">
       <hardware>
@@ -147,20 +152,36 @@
       <joint name="joint_1">
         <command_interface name="position"/>
-        <state_interface name="position"/>
+        <state_interface name="position">
+          <xacro:if value="${use_mock}">
+            <param name="initial_value">${initial_positions['joint_1']}</param>
+          </xacro:if>
+        </state_interface>
         <state_interface name="velocity"/>
       </joint>
       <joint name="joint_2">
         <command_interface name="position"/>
-        <state_interface name="position"/>
+        <state_interface name="position">
+          <xacro:if value="${use_mock}">
+            <param name="initial_value">${initial_positions['joint_2']}</param>
+          </xacro:if>
+        </state_interface>
         <state_interface name="velocity"/>
       </joint>
       <joint name="joint_3">
         <command_interface name="position"/>
-        <state_interface name="position"/>
+        <state_interface name="position">
+          <xacro:if value="${use_mock}">
+            <param name="initial_value">${initial_positions['joint_3']}</param>
+          </xacro:if>
+        </state_interface>
         <state_interface name="velocity"/>
       </joint>
       <joint name="joint_4">
         <command_interface name="position"/>
-        <state_interface name="position"/>
+        <state_interface name="position">
+          <xacro:if value="${use_mock}">
+            <param name="initial_value">${initial_positions['joint_4']}</param>
+          </xacro:if>
+        </state_interface>
         <state_interface name="velocity"/>
       </joint>
