Commit message: Joystick kind of works

File: src/my_arm_description/urdf/my_arm.urdf.xacro (robot description, xacro)
@@ -86,10 +86,10 @@
     </collision>
   </link>
-  <joint name="joint_1" type="revolute">
+  <joint name="joint_1" type="continuous">
     <parent link="base_link"/>
     <child link="link_1"/>
     <origin xyz="0 0 0.025" rpy="0 0 0"/>
     <axis xyz="0 0 1"/>
-    <limit lower="0.0" upper="6.283185" effort="100" velocity="1.0"/>
+    <limit effort="100" velocity="1.0"/>
   </joint>
   <joint name="joint_2" type="revolute">

File: src/my_arm_moveit_config/config/my_arm.ros2_control.xacro (robot description, xacro)
@@ -3,5 +3,5 @@
     <xacro:macro name="my_arm_ros2_control" params="name initial_positions_file use_mock_hardware">
         <xacro:property name="initial_positions" value="${load_yaml(initial_positions_file)['initial_positions']}"/>
-      <xacro:property name="use_mock" value="${use_mock_hardware}"/>
+        <xacro:property name="use_mock" value="${use_mock_hardware}"/>
         <ros2_control name="${name}" type="system">
             <hardware>
@@ -37,5 +37,7 @@
                 <command_interface name="position"/>
                 <state_interface name="position">
-                  <param name="initial_value">${initial_positions['joint_1']}</param>
+                  <xacro:if value="${use_mock}">
+                    <param name="initial_value">${initial_positions['joint_1']}</param>
+                  </xacro:if>
                 </state_interface>
                 <state_interface name="velocity"/>
@@ -44,5 +46,7 @@
                 <command_interface name="position"/>
                 <state_interface name="position">
-                  <param name="initial_value">${initial_positions['joint_2']}</param>
+                  <xacro:if value="${use_mock}">
+                    <param name="initial_value">${initial_positions['joint_2']}</param>
+                  </xacro:if>
                 </state_interface>
                 <state_interface name="velocity"/>
@@ -51,5 +55,7 @@
                 <command_interface name="position"/>
                 <state_interface name="position">
-                  <param name="initial_value">${initial_positions['joint_3']}</param>
+                  <xacro:if value="${use_mock}">
+                    <param name="initial_value">${initial_positions['joint_3']}</param>
+                  </xacro:if>
                 </state_interface>
                 <state_interface name="velocity"/>
@@ -58,5 +64,7 @@
                 <command_interface name="position"/>
                 <state_interface name="position">
-                  <param name="initial_value">${initial_positions['joint_4']}</param>
+                  <xacro:if value="${use_mock}">
+                    <param name="initial_value">${initial_positions['joint_4']}</param>
+                  </xacro:if>
                 </state_interface>
                 <state_interface name="velocity"/>
