Commit message: ros config changes

File: src/my_arm_description/urdf/my_arm.urdf.xacro (robot description, xacro)
@@ -1,7 +1,6 @@
 <?xml version="1.0"?>
 <robot xmlns:xacro="http://www.ros.org/wiki/xacro" name="my_arm">
-  <xacro:arg name="use_mock_hardware" default="false" />
-  <xacro:arg name="include_ros2_control" default="false" />
-  <xacro:property name="use_mock" value="$(arg use_mock_hardware)"/>
+  <!-- Kinematics only. ros2_control (mock or ESP32) is added by
+       my_arm_moveit_config/config/my_arm.ros2_control.xacro -->
   <material name="blue">
     <color rgba="0 0 0.8 1"/>
@@ -71,19 +70,6 @@
     </collision>
   </link>
-  <link name="link_4">
-    <visual>
-      <geometry>
-        <box size="0.05 0.05 0.05"/>
-      </geometry>
-      <origin xyz="0 0 0.025" rpy="0 0 0"/>
-      <material name="grey"/>
-    </visual>
-    <collision>
-      <geometry>
-        <box size="0.05 0.05 0.05"/>
-      </geometry>
-      <origin xyz="0 0 0.025" rpy="0 0 0"/>
-    </collision>
-  </link>
+  <!-- Tip of the forearm (no wrist yet). Used as the end effector for IK / Servo. -->
+  <link name="ee_link"/>
   <joint name="joint_1" type="continuous">
     <parent link="base_link"/>
@@ -107,63 +93,8 @@
     <limit lower="-3.141593" upper="0.0" effort="100" velocity="0.26"/>
   </joint>
-  <joint name="joint_4" type="revolute">
+  <joint name="ee_joint" type="fixed">
     <parent link="link_3"/>
-    <child link="link_4"/>
+    <child link="ee_link"/>
     <origin xyz="0 0 0.345" rpy="0 0 0"/>
-    <axis xyz="0 1 0"/>
-    <limit lower="-3.14" upper="3.14" effort="50" velocity="2.0"/>
   </joint>
-  <xacro:if value="$(arg include_ros2_control)">
-    <ros2_control name="MyRobotSystem" type="system">
-      <hardware>
-          <xacro:if value="${use_mock}">
-            <plugin>mock_components/GenericSystem</plugin>
-          </xacro:if>
-          <xacro:unless value="${use_mock}">
-            <plugin>my_arm_hardware/Esp32SerialHardware</plugin>
-            <param name="port">/dev/ttyUSB0</param>
-            <param name="baud_rate">115200</param>
-            <param name="real_joints">3</param>
-            <param name="id_offset">0</param>
-            <param name="query_period_ms">50</param>
-            <param name="poll_cur_ang">false</param>
-            <param name="stream_list_mode">true</param>
-            <param name="stream_without_id">false</param>
-            <param name="wait_for_first_state">true</param>
-            <param name="state_timeout_ms">1000</param>
-            <param name="ping_on_activate">true</param>
-            <param name="ping_id">50</param>
-            <param name="ping_timeout_ms">300</param>
-            <param name="joint_1_min_deg">0</param>
-            <param name="joint_1_max_deg">360</param>
-            <param name="joint_2_min_deg">0</param>
-            <param name="joint_2_max_deg">160</param>
-            <param name="joint_1_offset_deg">0</param>
-            <param name="joint_2_offset_deg">-90</param>
-            <param name="joint_3_offset_deg">-90</param>
-            <param name="joint_4_offset_deg">0</param>
-          </xacro:unless>
-      </hardware>
-      <joint name="joint_1">
-        <command_interface name="position"/>
-        <state_interface name="position"/>
-        <state_interface name="velocity"/>
-      </joint>
-      <joint name="joint_2">
-        <command_interface name="position"/>
-        <state_interface name="position"/>
-        <state_interface name="velocity"/>
-      </joint>
-      <joint name="joint_3">
-        <command_interface name="position"/>
-        <state_interface name="position"/>
-        <state_interface name="velocity"/>
-      </joint>
-      <joint name="joint_4">
-        <command_interface name="position"/>
-        <state_interface name="position"/>
-        <state_interface name="velocity"/>
-      </joint>
-    </ros2_control>
-  </xacro:if>
 </robot>

File: src/my_arm_moveit_config/config/my_arm.ros2_control.xacro (robot description, xacro)
@@ -31,5 +31,4 @@
             <param name="joint_2_offset_deg">-90</param>
             <param name="joint_3_offset_deg">-90</param>
-            <param name="joint_4_offset_deg">0</param>
           </xacro:unless>
             </hardware>
@@ -61,13 +60,4 @@
                 <state_interface name="velocity"/>
             </joint>
-            <joint name="joint_4">
-                <command_interface name="position"/>
-                <state_interface name="position">
-                  <xacro:if value="${use_mock}">
-                    <param name="initial_value">${initial_positions['joint_4']}</param>
-                  </xacro:if>
-                </state_interface>
-                <state_interface name="velocity"/>
-            </joint>
         </ros2_control>
     </xacro:macro>

Commit message: clean up

File: src/my_arm_description/urdf/my_arm.urdf.xacro (robot description, xacro)
@@ -84,5 +84,5 @@
     <origin xyz="0 0 0.1" rpy="0 0 0"/>
     <axis xyz="0 1 0"/>
-    <limit lower="-1.570796" upper="1.221730" effort="200" velocity="0.6"/>
+    <limit lower="-1.570796" upper="1.221730" effort="200" velocity="0.3"/>
   </joint>
   <joint name="joint_3" type="revolute">
@@ -91,5 +91,5 @@
     <origin xyz="0 0 0.405" rpy="0 0 0"/>
     <axis xyz="0 1 0"/>
-    <limit lower="-3.141593" upper="0.0" effort="100" velocity="0.26"/>
+    <limit lower="-2.792527" upper="0.0" effort="100" velocity="0.3"/>
   </joint>
   <joint name="ee_joint" type="fixed">

File: src/my_arm_moveit_config/config/my_arm.ros2_control.xacro (robot description, xacro)
@@ -1,5 +1,5 @@
 <?xml version="1.0"?>
 <robot xmlns:xacro="http://www.ros.org/wiki/xacro">
-    <xacro:macro name="my_arm_ros2_control" params="name initial_positions_file use_mock_hardware">
+    <xacro:macro name="my_arm_ros2_control" params="name initial_positions_file use_mock_hardware serial_port">
         <xacro:property name="initial_positions" value="${load_yaml(initial_positions_file)['initial_positions']}"/>
         <xacro:property name="use_mock" value="${use_mock_hardware}"/>
@@ -11,5 +11,5 @@
           <xacro:unless value="${use_mock}">
             <plugin>my_arm_hardware/Esp32SerialHardware</plugin>
-            <param name="port">/dev/ttyUSB0</param>
+            <param name="port">${serial_port}</param>
             <param name="baud_rate">115200</param>
                     <param name="real_joints">3</param>
@@ -24,8 +24,12 @@
                     <param name="ping_id">50</param>
             <param name="ping_timeout_ms">300</param>
-            <param name="joint_1_min_deg">0</param>
-            <param name="joint_1_max_deg">360</param>
+            <!-- Firmware angles (90 = straight up); must match the clamps in config.h -->
             <param name="joint_2_min_deg">0</param>
             <param name="joint_2_max_deg">160</param>
+            <param name="joint_3_min_deg">-70</param>
+            <param name="joint_3_max_deg">90</param>
+            <!-- Base: direction commands from the joystick (+1 right, -1 left, 0 stop) -->
+            <param name="base_cmd_topic">/base_cmd</param>
+            <param name="base_cmd_timeout_ms">200</param>
             <param name="joint_1_offset_deg">0</param>
             <param name="joint_2_offset_deg">-90</param>

File: src/my_arm_moveit_config/config/my_arm.urdf.xacro (robot description, xacro)
@@ -3,4 +3,7 @@
     <xacro:arg name="initial_positions_file" default="initial_positions.yaml" />
     <xacro:arg name="use_mock_hardware" default="false" />
+    <!-- ESP32 serial port. by-id path stays the same whichever ttyUSBn it gets. -->
+    <xacro:arg name="serial_port"
+               default="/dev/serial/by-id/usb-Silicon_Labs_CP2102_USB_to_UART_Bridge_Controller_0001-if00-port0" />
     <!-- Import my_arm urdf file -->
     <xacro:include filename="$(find my_arm_description)/urdf/my_arm.urdf.xacro" />
@@ -10,4 +13,5 @@
         name="FakeSystem"
         initial_positions_file="$(arg initial_positions_file)"
-        use_mock_hardware="$(arg use_mock_hardware)"/>
+        use_mock_hardware="$(arg use_mock_hardware)"
+        serial_port="$(arg serial_port)"/>
 </robot>
